File: 514_final_sensor_pcb/_autosave-514_final_sensor_pcb.kicad_sch (KiCad schematic)
At the start: 6 parts, among them SW1 SW_SPDT, U1 MOUDLE-SEEEDUINO-XIAO-ESP32C3

Commit message: sensor pcb v1.0
Parts:
- C1: value C -> 0.1uF
- R1: value R -> TBD
- R2: value PDV-P8103 -> TBT
Other:
- title: (none) -> Laura_Sensor_Board v1.0
- moved on the sheet: BT1, C1, R1, R2, SW1, U1
